File: kicad/teensy_motor_controller/teensy_motor_controller.kicad_sch (KiCad schematic)
At the start: 10 parts

Commit message: New functionality
Parts:
- removed J1: (no value), symbol Connector_Generic:Conn_01x11
- removed U1: (no value), symbol teensy_motor_controller-rescue:Teensy4.0-teensy
- added H1, H2, H3, H4: MountingHole, MountingHole:MountingHole_4.3mm_M4_Pad, symbol Mechanical:MountingHole
- added J1: 1869334, SamacSys_Parts:1869334, symbol SamacSys_Parts:1869334
- added J2: 1730162, SamacSys_Parts:1730162, symbol SamacSys_Parts:1730162
- added R5: R15k, Resistor_THT:R_Axial_DIN0207_L6.3mm_D2.5mm_P15.24mm_Horizontal, symbol Device:R
- added R6, R7: R10k, Resistor_THT:R_Axial_DIN0207_L6.3mm_D2.5mm_P15.24mm_Horizontal, symbol Device:R
- added R8: R5,5k, Resistor_THT:R_Axial_DIN0207_L6.3mm_D2.5mm_P15.24mm_Horizontal, symbol Device:R
- added U1: Teensy4.0_24pin, teensy:Teensy40_24pin, symbol teensy:Teensy4.0_24pin
- D1, D2, D3, D4: value (none) -> LED; footprint (none) -> LED_THT:LED_D5.0mm
- R1, R2, R3, R4: value (none) -> 220; footprint (none) -> Resistor_THT:R_Axial_DIN0207_L6.3mm_D2.5mm_P15.24mm_Horizontal
Connections:
- net X_max_led: now also U1.16 (16_A2_RX4_SCL1)
- net X_max_limit: now also J1.5, U1.8 (8_TX2_IN1)
- net X_min_led: now also U1.17 (17_A3_TX4_SDA1)
- net X_min_limit: now also J1.4, U1.9 (9_OUT1C)
- net X_stepper_direction: now also J1.9, U1.4 (4_BCLK2)
- net X_stepper_enable: now also J1.8, U1.5 (5_IN2)
- net X_stepper_pulse: now also J1.10, U1.3 (3_LRCLK2)
- net Z_max_led: now also U1.14 (14_A0_TX3_SPDIF_OUT)
- net Z_max_limit: now also J1.7, U1.6 (6_OUT1D)
- net Z_min_led: now also U1.15 (15_A1_RX3_SPDIF_IN)
- net Z_min_limit: now also J1.6, U1.7 (7_RX2_OUT1A)
- net Z_stepper_direction: now also J1.12, U1.1 (1_TX1_CTX2_MISO1)
- net Z_stepper_enable: now also J1.11, U1.2 (2_OUT2)
- net Z_stepper_pulse: now also J1.13, U1.0 (0_RX1_CRX2_CS1)
- net at R1.1, R2.1, R3.1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: now also J1.14, U1.GND1 (GND)
- new net: R8.1, U1.GND2 (0_RX1_CRX2_CS1)
- new net: R5.2, R8.2, U1.18 (18_A4_SDA0)
- new net: J1.1, U1.12 (12_MISO_MQSL)
- new net: J1.2, U1.11 (11_MOSI_CTX1)
- new net: J1.3, U1.10 (10_CS_MQSR)
- new net: J2.2, U1.19 (19_A5_SCL0)
- new net: J2.3, U1.20 (20_A6_TX5_LRCLK1)
- new net: J2.4, U1.21 (21_A7_RX5_BCLK1)
- new net: J2.5, U1.22 (22_A8_CTX1)
- new net: J2.6, U1.23 (23_A9_CRX1_MCLK1)
- new net: J2.1, R7.2
- new net: R5.1, R6.1
- new net: R6.2, R7.1
- no-connect marks 39 -> 1
Other:
- moved on the sheet: R1, R2, R3, R4
